Commit message: <feat> add basic import of AAR
1. add dragon
2. add spidar

File: source/aerial_lab/data/Robots/dragon/dragon.urdf (robot description, URDF)
Before this commit: robot dragon, 29 links, 28 joints
Joints:
- joint rotor1: limit lower=2 upper=30 effort=100.0 velocity=0.5 -> effort=100.0 velocity=0.5
- joint rotor2: limit lower=2 upper=30 effort=100.0 velocity=0.5 -> effort=100.0 velocity=0.5
- joint rotor3: limit lower=2 upper=30 effort=100.0 velocity=0.5 -> effort=100.0 velocity=0.5
- joint rotor4: limit lower=2 upper=30 effort=100.0 velocity=0.5 -> effort=100.0 velocity=0.5

File: source/aerial_lab/data/Robots/spidar/spidar_v1_leg.urdf (robot description, URDF)
Before this commit: robot spidar, 80 links, 79 joints
Links:
- link bat1: geometry visual mesh filename=package://spidar/mesh/battery/ZIPPY_3000_25C_6S.dae
- link bat2: geometry visual mesh filename=package://spidar/mesh/battery/ZIPPY_3000_25C_6S.dae
- link bat3: geometry visual mesh filename=package://spidar/mesh/battery/ZIPPY_3000_25C_6S.dae
- link bat4: geometry visual mesh filename=package://spidar/mesh/battery/ZIPPY_3000_25C_6S.dae
- link bat5: geometry visual mesh filename=package://spidar/mesh/battery/ZIPPY_3000_25C_6S.dae
- link bat6: geometry visual mesh filename=package://spidar/mesh/battery/ZIPPY_3000_25C_6S.dae
- link bat7: geometry visual mesh filename=package://spidar/mesh/battery/ZIPPY_3000_25C_6S.dae
- link bat8: geometry visual mesh filename=package://spidar/mesh/battery/ZIPPY_3000_25C_6S.dae

File: source/aerial_lab/data/Robots/spidar/spidar_v1_leg_stl.urdf (robot description, URDF)
Before this commit: robot spidar, 80 links, 79 joints
Links:
- removed link end_leg2
- removed link end_leg4
- removed link end_leg6
- removed link end_leg8
- added link link2_foot, mass 0.09; collision sphere radius=0.04; visual mesh filename=package://spidar/mesh/leg/leg_cap.stl
- added link link4_foot, mass 0.09; collision sphere radius=0.04; visual mesh filename=package://spidar/mesh/leg/leg_cap.stl
- added link link6_foot, mass 0.09; collision sphere radius=0.04; visual mesh filename=package://spidar/mesh/leg/leg_cap.stl
- added link link8_foot, mass 0.09; collision sphere radius=0.04; visual mesh filename=package://spidar/mesh/leg/leg_cap.stl
- link bat1: geometry visual mesh filename=package://spidar/mesh/battery/ZIPPY_3000_25C_6S.stl
- link bat2: geometry visual mesh filename=package://spidar/mesh/battery/ZIPPY_3000_25C_6S.stl
- link bat3: geometry visual mesh filename=package://spidar/mesh/battery/ZIPPY_3000_25C_6S.stl
- link bat4: geometry visual mesh filename=package://spidar/mesh/battery/ZIPPY_3000_25C_6S.stl
- link bat5: geometry visual mesh filename=package://spidar/mesh/battery/ZIPPY_3000_25C_6S.stl
- link bat6: geometry visual mesh filename=package://spidar/mesh/battery/ZIPPY_3000_25C_6S.stl
- link bat7: geometry visual mesh filename=package://spidar/mesh/battery/ZIPPY_3000_25C_6S.stl
- link bat8: geometry visual mesh filename=package://spidar/mesh/battery/ZIPPY_3000_25C_6S.stl
- link center_link: geometry collision cylinder length=0.0928 radius=0.169; visual mesh filename=package://spidar/mesh/link/center_link.stl
- link fc: geometry visual mesh filename=package://spidar/mesh/board/spinal.stl
- link gimbal1_pitch_module: geometry visual mesh filename=package://spidar/mesh/link/pitch_link.stl
- link gimbal1_roll_module: geometry visual mesh filename=package://spidar/mesh/link/roll_link.stl
- link gimbal2_pitch_module: geometry visual mesh filename=package://spidar/mesh/link/pitch_link.stl
- link gimbal2_roll_module: geometry visual mesh filename=package://spidar/mesh/link/roll_link.stl
- link gimbal3_pitch_module: geometry visual mesh filename=package://spidar/mesh/link/pitch_link.stl
- link gimbal3_roll_module: geometry visual mesh filename=package://spidar/mesh/link/roll_link.stl
- link gimbal4_pitch_module: geometry visual mesh filename=package://spidar/mesh/link/pitch_link.stl
- link gimbal4_roll_module: geometry visual mesh filename=package://spidar/mesh/link/roll_link.stl
- link gimbal5_pitch_module: geometry visual mesh filename=package://spidar/mesh/link/pitch_link.stl
- link gimbal5_roll_module: geometry visual mesh filename=package://spidar/mesh/link/roll_link.stl
- link gimbal6_pitch_module: geometry visual mesh filename=package://spidar/mesh/link/pitch_link.stl
- link gimbal6_roll_module: geometry visual mesh filename=package://spidar/mesh/link/roll_link.stl
- link gimbal7_pitch_module: geometry visual mesh filename=package://spidar/mesh/link/pitch_link.stl
- link gimbal7_roll_module: geometry visual mesh filename=package://spidar/mesh/link/roll_link.stl
- link gimbal8_pitch_module: geometry visual mesh filename=package://spidar/mesh/link/pitch_link.stl
- link gimbal8_roll_module: geometry visual mesh filename=package://spidar/mesh/link/roll_link.stl
- link joint_junction_leg1: geometry collision cylinder length=0.1045 radius=0.01; visual mesh filename=package://spidar/mesh/leg/long_leg.stl
- link joint_junction_leg2: geometry collision cylinder length=0.1045 radius=0.01; visual mesh filename=package://spidar/mesh/leg/long_leg.stl
- link joint_junction_leg3: geometry collision cylinder length=0.1045 radius=0.01; visual mesh filename=package://spidar/mesh/leg/long_leg.stl
- link joint_junction_leg4: geometry collision cylinder length=0.1045 radius=0.01; visual mesh filename=package://spidar/mesh/leg/long_leg.stl
- link joint_junction_leg5: geometry collision cylinder length=0.1045 radius=0.01; visual mesh filename=package://spidar/mesh/leg/long_leg.stl
- link joint_junction_leg6: geometry collision cylinder length=0.1045 radius=0.01; visual mesh filename=package://spidar/mesh/leg/long_leg.stl
- link joint_junction_leg7: geometry collision cylinder length=0.1045 radius=0.01; visual mesh filename=package://spidar/mesh/leg/long_leg.stl
- link joint_junction_leg8: geometry collision cylinder length=0.1045 radius=0.01; visual mesh filename=package://spidar/mesh/leg/long_leg.stl
- link joint_junction_link2: geometry visual mesh filename=package://spidar/mesh/link/joint_junction_link.stl
- link joint_junction_link4: geometry visual mesh filename=package://spidar/mesh/link/joint_junction_link.stl
- link joint_junction_link6: geometry visual mesh filename=package://spidar/mesh/link/joint_junction_link.stl
- link joint_junction_link8: geometry visual mesh filename=package://spidar/mesh/link/joint_junction_link.stl
- link link1: geometry collision cylinder length=0.523 radius=0.025; visual mesh filename=package://spidar/mesh/link/general_link.stl
- link link2: geometry collision cylinder length=0.523 radius=0.025; visual mesh filename=package://spidar/mesh/link/end_link.stl
- link link3: geometry collision cylinder length=0.523 radius=0.025; visual mesh filename=package://spidar/mesh/link/general_link.stl
- link link4: geometry collision cylinder length=0.523 radius=0.025; visual mesh filename=package://spidar/mesh/link/end_link.stl
- link link5: geometry collision cylinder length=0.523 radius=0.025; visual mesh filename=package://spidar/mesh/link/general_link.stl
- link link6: geometry collision cylinder length=0.523 radius=0.025; visual mesh filename=package://spidar/mesh/link/end_link.stl
- link link7: geometry collision cylinder length=0.523 radius=0.025; visual mesh filename=package://spidar/mesh/link/general_link.stl
- link link8: geometry collision cylinder length=0.523 radius=0.025; visual mesh filename=package://spidar/mesh/link/end_link.stl
- link pc: mass 0.1411331 -> 0.096; geometry visual mesh filename=package://spidar/mesh/board/vim4_module.stl
Joints:
- removed joint link22end_leg2
- removed joint link42end_leg4
- removed joint link62end_leg6
- removed joint link82end_leg8
- added joint link22link2_foot: type fixed, parent link2, child link2_foot, origin xyz=0.5115 0 0 rpy=0 0 0, axis 0 0 1, limit lower=0 upper=0 effort=100 velocity=100
- added joint link42link4_foot: type fixed, parent link4, child link4_foot, origin xyz=0.5115 0 0 rpy=0 0 0, axis 0 0 1, limit lower=0 upper=0 effort=100 velocity=100
- added joint link62link6_foot: type fixed, parent link6, child link6_foot, origin xyz=0.5115 0 0 rpy=0 0 0, axis 0 0 1, limit lower=0 upper=0 effort=100 velocity=100
- added joint link82link8_foot: type fixed, parent link8, child link8_foot, origin xyz=0.5115 0 0 rpy=0 0 0, axis 0 0 1, limit lower=0 upper=0 effort=100 velocity=100
- joint center_link2pc: origin xyz=0 0.089888 0.002 rpy=1.5707963267948966 0 0 -> xyz=0 0 -0.047 rpy=0 0 0

File: source/aerial_lab/data/Robots/spidar/urdf/link.urdf.xacro (robot description, xacro)
@@ -305,5 +305,5 @@
     <xacro:if value="${battery == 1}">
       <xacro:extra_module name="bat${self}" parent="link${self}" visible="1"
-                          model_url="package://spidar/mesh/battery/ZIPPY-3000-25C-6S.dae">
+                          model_url="package://spidar/mesh/battery/ZIPPY_3000_25C_6S.dae">
         <xacro:if value="${link_type == 'general'}">
           <origin xyz="0.430 0.0 -0.039" rpy="${-pi/2} 0 0"/>
