Commit message: <feat> add force visualization and rotor.py
1. add force visualization with contact sensor
2. modify spidar `.urdf` for proper import
3. add rotor.py but not tested

File: source/aerial_lab/data/Robots/spidar/spidar_v1_leg_stl.urdf (robot description, URDF)
Before this commit: robot spidar, 80 links, 79 joints
Links:
- link link2: geometry collision cylinder length=0.403 radius=0.025; visual mesh filename=package://spidar/mesh/link/end_link.stl
- link link4: geometry collision cylinder length=0.403 radius=0.025; visual mesh filename=package://spidar/mesh/link/end_link.stl
- link link6: geometry collision cylinder length=0.403 radius=0.025; visual mesh filename=package://spidar/mesh/link/end_link.stl
- link link8: geometry collision cylinder length=0.403 radius=0.025; visual mesh filename=package://spidar/mesh/link/end_link.stl
