Commit message: <feat> add robot in rl_env
1. modify .urdf to meet isaaclab's urdf importer
2. try to add {contact sensor, rotor, motor} to beetle from quadcopter
3. try to add {contact sensor, rotor, motor} to beetle from template

File: source/aerial_lab/data/Robots/beetle/beetle.urdf (robot description, URDF)
Before this commit: robot beetle, 23 links, 22 joints
Links:
- link base_link: geometry collision box size=0.52 0.52 0.241; visual mesh filename=package://beetle/mesh/base_link_beetle_art.dae
Joints:
- joint dummy_arm_palm_joint: axis 1 0 0 -> (none); limit lower=0 upper=0 effort=0 velocity=0 -> (none); type revolute -> fixed
- joint dummy_palm_gripper_joint: axis 1 0 0 -> (none); limit lower=0 upper=0 effort=0 velocity=0 -> (none); type revolute -> fixed
- joint rotor1: limit lower=1.0 upper=30.0 effort=100.0 velocity=0.5 -> effort=100.0 velocity=0.5
- joint rotor2: limit lower=1.0 upper=30.0 effort=100.0 velocity=0.5 -> effort=100.0 velocity=0.5
- joint rotor3: limit lower=1.0 upper=30.0 effort=100.0 velocity=0.5 -> effort=100.0 velocity=0.5
- joint rotor4: limit lower=1.0 upper=30.0 effort=100.0 velocity=0.5 -> effort=100.0 velocity=0.5

File: source/aerial_lab/data/Robots/beetle_omni/beetle_art_omni.urdf (robot description, URDF)
Before this commit: robot beetle-art-omni, 22 links, 21 joints
Joints:
- joint rotor1: limit lower=1.0 upper=30.0 effort=100.0 velocity=0.5 -> effort=100.0 velocity=0.5
- joint rotor2: limit lower=1.0 upper=30.0 effort=100.0 velocity=0.5 -> effort=100.0 velocity=0.5
- joint rotor3: limit lower=1.0 upper=30.0 effort=100.0 velocity=0.5 -> effort=100.0 velocity=0.5
- joint rotor4: limit lower=1.0 upper=30.0 effort=100.0 velocity=0.5 -> effort=100.0 velocity=0.5

Commit message: <feat> make smallest demonstration of (A)rticulated-(A)erial-(R)obotics
1. aerial_beetle_env is smallest AAR env
2. modify .ursd files for correct visualization (rotor rotation)
3. perf vscode configuration files

File: source/aerial_lab/data/Robots/beetle/beetle.urdf (robot description, URDF)
Before this commit: robot beetle, 23 links, 22 joints
Links:
- link gimbal_link1: geometry collision cylinder length=0.033 radius=0.02
- link gimbal_link2: geometry collision cylinder length=0.033 radius=0.02
- link gimbal_link3: geometry collision cylinder length=0.033 radius=0.02
- link gimbal_link4: geometry collision cylinder length=0.033 radius=0.02
- link thrust1: geometry visual mesh filename=package://beetle/mesh/prop_5inch.dae
- link thrust2: geometry visual mesh filename=package://beetle/mesh/prop_5inch.dae
- link thrust3: geometry visual mesh filename=package://beetle/mesh/prop_5inch.dae
- link thrust4: geometry visual mesh filename=package://beetle/mesh/prop_5inch.dae
Joints:
- joint rotor1: limit effort=100.0 velocity=0.5 -> effort=100.0 velocity=25.0
- joint rotor2: limit effort=100.0 velocity=0.5 -> effort=100.0 velocity=25.0
- joint rotor3: limit effort=100.0 velocity=0.5 -> effort=100.0 velocity=25.0
- joint rotor4: limit effort=100.0 velocity=0.5 -> effort=100.0 velocity=25.0

Commit message: <save> beetle ideal pose env, ood to position tracking with zero RPY
1. modify beetle.urdf for correct visualization
2. try to find a proper way to train pose controller

File: source/aerial_lab/data/Robots/beetle/beetle.urdf (robot description, URDF)
Before this commit: robot beetle, 23 links, 22 joints
Links:
- link base_link: geometry collision box size=0.52 0.52 0.241; visual mesh filename=package://beetle/mesh/base_link_hyper.dae
- link gimbal_link1: geometry collision cylinder length=0.033 radius=0.02; visual mesh filename=package://beetle/mesh/rotor_module.dae
- link gimbal_link2: geometry collision cylinder length=0.033 radius=0.02; visual mesh filename=package://beetle/mesh/rotor_module.dae
- link gimbal_link3: geometry collision cylinder length=0.033 radius=0.02; visual mesh filename=package://beetle/mesh/rotor_module.dae
- link gimbal_link4: geometry collision cylinder length=0.033 radius=0.02; visual mesh filename=package://beetle/mesh/rotor_module.dae
- link thrust1: geometry 
- link thrust2: geometry 
- link thrust3: geometry 
- link thrust4: geometry 

File: source/aerial_lab/data/Robots/spidar/spidar_v1_leg.urdf (robot description, URDF)
Before this commit: robot spidar, 80 links, 79 joints
Links:
- link edf1_left: geometry collision cylinder length=0.065 radius=0.085
- link edf1_right: geometry collision cylinder length=0.065 radius=0.085
- link edf2_left: geometry collision cylinder length=0.065 radius=0.085
- link edf2_right: geometry collision cylinder length=0.065 radius=0.085
- link edf3_left: geometry collision cylinder length=0.065 radius=0.085
- link edf3_right: geometry collision cylinder length=0.065 radius=0.085
- link edf4_left: geometry collision cylinder length=0.065 radius=0.085
- link edf4_right: geometry collision cylinder length=0.065 radius=0.085
- link edf5_left: geometry collision cylinder length=0.065 radius=0.085
- link edf5_right: geometry collision cylinder length=0.065 radius=0.085
- link edf6_left: geometry collision cylinder length=0.065 radius=0.085
- link edf6_right: geometry collision cylinder length=0.065 radius=0.085
- link edf7_left: geometry collision cylinder length=0.065 radius=0.085
- link edf7_right: geometry collision cylinder length=0.065 radius=0.085
- link edf8_left: geometry collision cylinder length=0.065 radius=0.085
- link edf8_right: geometry collision cylinder length=0.065 radius=0.085
- link link2: geometry collision cylinder length=0.423 radius=0.025; visual mesh filename=package://spidar/mesh/link/end_link.dae
- link link4: geometry collision cylinder length=0.423 radius=0.025; visual mesh filename=package://spidar/mesh/link/end_link.dae
- link link6: geometry collision cylinder length=0.423 radius=0.025; visual mesh filename=package://spidar/mesh/link/end_link.dae
- link link8: geometry collision cylinder length=0.423 radius=0.025; visual mesh filename=package://spidar/mesh/link/end_link.dae

File: source/aerial_lab/data/Robots/spidar/spidar_v1_leg_stl.urdf (robot description, URDF)
Before this commit: robot spidar, 80 links, 79 joints
Links:
- link edf1_left: geometry collision cylinder length=0.065 radius=0.085
- link edf1_right: geometry collision cylinder length=0.065 radius=0.085
- link edf2_left: geometry collision cylinder length=0.065 radius=0.085
- link edf2_right: geometry collision cylinder length=0.065 radius=0.085
- link edf3_left: geometry collision cylinder length=0.065 radius=0.085
- link edf3_right: geometry collision cylinder length=0.065 radius=0.085
- link edf4_left: geometry collision cylinder length=0.065 radius=0.085
- link edf4_right: geometry collision cylinder length=0.065 radius=0.085
- link edf5_left: geometry collision cylinder length=0.065 radius=0.085
- link edf5_right: geometry collision cylinder length=0.065 radius=0.085
- link edf6_left: geometry collision cylinder length=0.065 radius=0.085
- link edf6_right: geometry collision cylinder length=0.065 radius=0.085
- link edf7_left: geometry collision cylinder length=0.065 radius=0.085
- link edf7_right: geometry collision cylinder length=0.065 radius=0.085
- link edf8_left: geometry collision cylinder length=0.065 radius=0.085
- link edf8_right: geometry collision cylinder length=0.065 radius=0.085
- link link2: geometry collision cylinder length=0.423 radius=0.025; visual mesh filename=package://spidar/mesh/link/end_link.stl
- link link4: geometry collision cylinder length=0.423 radius=0.025; visual mesh filename=package://spidar/mesh/link/end_link.stl
- link link6: geometry collision cylinder length=0.423 radius=0.025; visual mesh filename=package://spidar/mesh/link/end_link.stl
- link link8: geometry collision cylinder length=0.423 radius=0.025; visual mesh filename=package://spidar/mesh/link/end_link.stl
