Commit message: <feat> try delayed joint cmd and angle target

File: source/aerial_lab/data/Robots/beetle_hyper/beetle_hyper.urdf (robot description, URDF)
Before this commit: robot gimbalrotor, 19 links, 18 joints
Joints:
- joint gimbal1: limit lower=-1.57 upper=1.57 effort=6.6 velocity=3.0 -> lower=-3.926991 upper=3.926991 effort=6.6 velocity=3.0
- joint gimbal2: limit lower=-1.57 upper=1.57 effort=6.6 velocity=3.0 -> lower=-3.926991 upper=3.926991 effort=6.6 velocity=3.0
- joint gimbal3: limit lower=-1.57 upper=1.57 effort=6.6 velocity=3.0 -> lower=-3.926991 upper=3.926991 effort=6.6 velocity=3.0
- joint gimbal4: limit lower=-1.57 upper=1.57 effort=6.6 velocity=3.0 -> lower=-3.926991 upper=3.926991 effort=6.6 velocity=3.0
