Commit message: <feat|log:2025-12-10_14-34-50>
1. add samplecenter
2. add orientation guided thrust_uneven
3. add MiniQuadcopter env
4. correct some typo

File: source/aerial_lab/data/Robots/mini_quadrotor/mini_quadrotor.urdf (robot description, URDF)
Before this commit: robot module_quadrotor, 9 links, 8 joints
Links:
- removed link main_body
- added link base_link, mass 0.832; collision box size=0.32 0.32 0.16; visual mesh filename=package://mini_quadrotor/mesh/main_body_livox.dae
- link fc: mass 00 -> 0.00001
- link lidar_imu: mass 00 -> 0.00001
Joints:
- joint main_body2battery: parent main_body -> base_link
- joint main_body2fc: parent main_body -> base_link
- joint main_body2lidar_imu: parent main_body -> base_link
- joint root_joint: child main_body -> base_link
- joint rotor1: parent main_body -> base_link
- joint rotor2: parent main_body -> base_link
- joint rotor3: parent main_body -> base_link
- joint rotor4: parent main_body -> base_link
